File: LMD18200.kicad_sch (KiCad schematic)
At the start: 5 parts, among them J4 Conn_01x02_Socket, U2 LMD18200

Commit message: First Commit , BOM
Parts:
- C4, C5: LCSC# (none) -> C57112
- R3: LCSC# (none) -> C2907113
- U2: LCSC# (none) -> C117011
