File: motorBoardCan.kicad_sch (KiCad schematic)
At the start: 21 parts, among them J1 Conn_01x04_Pin, J2 Conn_01x04_Pin, J3 Conn_02x04_Top_Bottom, J6 Conn_02x04_Top_Bottom, U1 NUCLEO-G431KB, U4 SN65HVD230, U5 LD1117S33TR_SOT223

Commit message: First Commit , BOM
Parts:
- C1, C3: LCSC# (none) -> C29823
- C2: LCSC# (none) -> C91151
- C6: LCSC# (none) -> C398835
- C7: value 10µF -> 10uF; LCSC# (none) -> C1713
- D1: footprint Diode_SMD:D_1206_3216Metric -> Capacitor_SMD:C_0805_2012Metric; LCSC# (none) -> C118721
- F1: LCSC# (none) -> C27515
- J1, J2: LCSC# (none) -> C2691448
- J3, J6: LCSC# (none) -> C277661
- R1: LCSC# (none) -> C2907128
- R6: LCSC# (none) -> C21189
- U1: Availability In Stock -> (none); Check_prices https://www.snapeda.com/parts/NUCLEO-G431KB/STMicroelectron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 -> (none); DESCRIPTION STM32F303K8, mbed-Enabled Development Nucleo-32 STM32F3 ARM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 -> (none); DIGI-KEY_PART_NUMBER 497-15981-ND -> (none); Description_1 STM32G431 Nucleo-32 STM32G4 ARM® Cortex®-M4 MCU 32-Bit Embe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 -> (none); MF STMicroelectronics -> (none); MP NUCLEO-G431KB -> (none); PACKAGE None -> (none); PURCHASE-URL https://pricing.snapeda.com/search/part/NUCLEO-F303K8/?ref=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 -> (none); Package None -> (none); Price None -> (none); SnapEDA_Link https://www.snapeda.com/parts/NUCLEO-G431KB/STMicroelectron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 -> (none)
- U4: LCSC# (none) -> C12084
- U5: LCSC# (none) -> C20538890
