File: motorBoardCan.kicad_pcb (KiCad board)
At the start: 6 copper layers, 50 x 50 mm, 46 parts, among them J1 Conn_01x04_Pin, J2 Conn_01x04_Pin, J3 Conn_02x04_Top_Bottom, J4 Conn_01x02_Socket, J5 Conn_01x02_Socket, J6 Conn_02x04_Top_Bottom, U1 NUCLEO-G431KB, U10 TPS563200, U2 LMD18200, U4 SN65HVD230, U5 LD1117S33TR_SOT223, U6 LMD18200

Commit message: Add BOM
Parts:
- removed ?: , 
- added H3: MountingHole, LibraryVictor:MountingHole_3.2mm_M3, F.Cu at (123.8, 104.0)
- C21, C24: footprint LED_SMD:LED_0805_2012Metric -> Capacitor_SMD:C_0805_2012Metric
- C22, C25: footprint Capacitor_SMD:C_1206_3216Metric -> Capacitor_SMD:C_0805_2012Metric
- C7: value 10µF -> 10uF
- D1: footprint Diode_SMD:D_1206_3216Metric -> Capacitor_SMD:C_0805_2012Metric
- D4: value LED_Small -> LED_G
- R4: value 220R -> 2kR
